Commit message: Added vesc node which converts to the real commands to send over the line. Cleaned up a bit

File: src/snail_description/urdf/snail.urdf.xacro (robot description, xacro)
@@ -135,5 +135,9 @@
     <child  link="rear_steer_link"/>
     <origin xyz="${rear_axle_x} 0 ${ground_clearance}" rpy="0 0 0"/>
-    <axis xyz="0 0 1"/>
+    <!-- Axis inverted (0 0 -1) so that positive joint angle matches positive
+         angular.z from the front-steer-assuming tricycle_steering_controller.
+         The deprecated front_steering:=false param used to handle this; we do
+         it geometrically instead. -->
+    <axis xyz="0 0 -1"/>
     <limit lower="${-steer_limit}" upper="${steer_limit}" effort="40.0" velocity="2.0"/>
     <dynamics damping="0.5" friction="0.0"/>
